File: Kicad/attiny2313_tm1637_ds1302/attiny2313_tm1637_ds1302.sch (KiCad schematic (older format))
At the start: 4 parts

Commit message: fix BYTE number register
Parts:
- added BT1: Battery_Cell, Battery:BatteryHolder_Keystone_103_1x20mm, symbol Device:Battery_Cell
- added BZ1: Buzzer, Buzzer_Beeper:Buzzer_12x9.5RM7.6, symbol Device:Buzzer
- added D1, D2: DIODE, Diode_THT:D_DO-15_P12.70mm_Horizontal, symbol Simulation_SPICE:DIODE
- added Q1: S9014, Package_TO_SOT_THT:TO-39-3, symbol Transistor_BJT:2N2219
- added R1, R2: 10kOm, Resistor_THT:R_Axial_DIN0309_L9.0mm_D3.2mm_P12.70mm_Horizontal, symbol Device:R
- added R3: R_Variable, Potentiometer_THT:Potentiometer_Vishay_T73YP_Vertical, symbol Device:R_Variable
- added SW_1: Mode, Button_Switch_THT:SW_PUSH_6mm, symbol Switch:SW_Push
- added SW_2: Clock_mode, Button_Switch_THT:SW_PUSH_6mm, symbol Switch:SW_Push
- added SW_3: Brightness, Button_Switch_THT:SW_PUSH_6mm, symbol Switch:SW_Push
- U3: renamed from U?; footprint (none) -> Module:tm1637-module; symbol Display_Graphic:tm1637-module -> attiny2313_tm1637_ds1302-rescue:tm1637-module-Display_Graphic
- Y1: renamed from Y?; footprint (none) -> Crystal:Crystal_AT310_D3.0mm_L10.0mm_Vertical
- gave numbers to parts that had none: 2
Connections:
- net labels added: CLK, DIO, GND, I\O, RST, SCLK, VCC
- wire segments 4 -> 46
- no-connect marks 0 -> 10

Commit message: created PCB
Parts:
- removed BT1: Battery_Cell, Battery:BatteryHolder_Keystone_103_1x20mm, symbol Device:Battery_Cell
- added J1: Conn_01x02, Battery:power_pins_smd, symbol Connector_Generic:Conn_01x02
- added J2, J3: Conn_01x04, Connector:conn_01x04, symbol Connector_Generic:Conn_01x04
- D1, D2: footprint Diode_THT:D_DO-15_P12.70mm_Horizontal -> Diode_THT:D_DO-15_P3.81mm_Vertical_KathodeUp
- Q1: footprint Package_TO_SOT_THT:TO-39-3 -> Package_TO_SOT_THT:SIPAK_Vertical
- R1, R2: footprint Resistor_THT:R_Axial_DIN0309_L9.0mm_D3.2mm_P12.70mm_Horizontal -> Resistor_THT:R_Axial_DIN0309_L9.0mm_D3.2mm_P5.08mm_Vertical
- U3: symbol attiny2313_tm1637_ds1302-rescue:tm1637-module-Display_Graphic -> attiny2313_tm1637_ds1302-rescue:tm1637-module-Display_Graphic-attiny2313_tm1637_ds1302-rescue
Connections:
- net labels removed: CLK, DIO
- wire segments 46 -> 66
Other:
- moved on the sheet: BZ1, D1, D2, Q1, R1, R2, R3, SW_1, SW_2, SW_3, U1, U2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

Commit message: убрана регулировка яркости, убрана кнопка яркости
Parts:
- removed D1, D2: DIODE, Diode_THT:D_DO-15_P3.81mm_Vertical_KathodeUp, symbol Simulation_SPICE:DIODE
- removed R3: R_Variable, Potentiometer_THT:Potentiometer_Vishay_T73YP_Vertical, symbol Device:R_Variable
- removed SW_2: Clock_mode, Button_Switch_THT:SW_PUSH_6mm, symbol Switch:SW_Push
- removed U3: tm1637-module, Module:tm1637-module, symbol attiny2313_tm1637_ds1302-rescue:tm1637-module-Display_Graphic-attiny2313_tm1637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
- added J4: Conn_01x04, Connector:conn_01x04, symbol Connector_Generic:Conn_01x04
- added RV1: R_POT, Potentiometer_THT:Potentiometer_Bourns_3386P_Vertical, symbol Device:R_POT
- Q1: footprint Package_TO_SOT_THT:SIPAK_Vertical -> Package_TO_SOT_THT:TO-92_Inline
- R1, R2: footprint Resistor_THT:R_Axial_DIN0309_L9.0mm_D3.2mm_P5.08mm_Vertical -> Resistor_THT:R_Axial_DIN0204_L3.6mm_D1.6mm_P5.08mm_Horizontal
- SW_2: renamed from SW_3; value Brightness -> Clock_Set
- U2: symbol Timer_RTC:DS1302+ -> attiny2313_tm1637_ds1302-rescue:DS1302+-Timer_RTC
- Y1: footprint Crystal:Crystal_AT310_D3.0mm_L10.0mm_Vertical -> Crystal:Crystal_C26-LF_D2.1mm_L6.5mm_Horizontal
Connections:
- net GND: now also J4.3 (Pin_3), RV1.2
- net I\O: now also U1.16 (PB4); no longer U1.17 (PB5)
- net RST: now also U1.17 (PB5); no longer U1.15 (PB3)
- net SCLK: now also U1.15 (PB3); no longer U1.16 (PB4)
- net at U1.12 (PB0): now also J4.2 (Pin_2)
- net at U1.13 (PB1): now also J4.1 (Pin_1)
- net at BZ1.1 (-), J1.1 (Pin_1), R1.1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: now also U2.1 (VCC2), J4.4 (Pin_4)
- net at U1.7 (PD3): now also J2.2 (Pin_2); no longer J2.3 (Pin_3)
- net at Q1.1 (E): now also RV1.1
- no-connect marks 10 -> 11
Other:
- moved on the sheet: BZ1, J1, J2, J3, Q1, R1, R2, SW_1, SW_2, U1, U2, Y1
